File: PCB/Diom-34SP_PCB/Diom-34SP_PCB.kicad_pcb (KiCad board)
At the start: 2 copper layers, 133.5 x 101.1 mm, 29 parts, among them J1 Conn_01x02_Male, U1 nice_nano

Commit message: Added On/Off Switch
Parts:
- added SW1: SHOU_HAN_MSK12C02-HB, led:SHOU HAN MSK12C02-HB, B.Cu at (186.5, 88.9)
Connections:
- J1 pad 2: B+ -> Net-(J1-Pad2)
Routing:
- net Net-(J1-Pad2): track 0.00 -> 4.23 mm
- net B+: track 50.5 -> 49.2 mm
Changed lines of the file:
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@@
   (net 26 "MX16")
   (net 27 "MX17")
+  (net 28 "Net-(J1-Pad2)")
+  (net 29 "unconnected-(SW1-Pad1)")
   (footprint "mx-switches-doubleSided:CherryMX-1U-doubleSided" (layer "F.Cu")
     (at 106.3625 50.8)
@@
       (net 8 "B-") (pinfunction "Pin_1") (pintype "passive"))
     (pad "2" thru_hole oval (at 2.5 0) (size 1.7 2) (drill 1) (layers *.Cu *.Mask)
-      (net 9 "B+") (pinfunction "Pin_2") (pintype "passive"))
+      (net 28 "Net-(J1-Pad2)") (pinfunction "Pin_2") (pintype "passive"))
     (model "${KICAD6_3DMODEL_DIR}/Connector_JST.3dshapes/JST_EH_S2B-EH_1x02_P2.50mm_Horizontal.wrl"
       (offset (xyz 0 0 0))
@@
     (pad "" np_thru_hole circle (at 0 0) (size 2.2 2.2) (drill 2.2) (layers *.Cu *.Mask))
   )
+  (footprint "led:SHOU HAN MSK12C02-HB" (layer "B.Cu")
+    (at 186.53125 88.9 -90)
+    (property "Sheetfile" "Diom-34SP_PCB.kicad_sch")
+    (property "Sheetname" "")
+    (attr smd)
+    (fp_text reference "SW1" (at -5.6 0 unlocked) (layer "B.SilkS")
+      (effects (font (size 1 1) (thickness 0.15)) (justify mirror))
+    )
+    (fp_text value "SHOU_HAN_MSK12C02-HB" (at 0 -2.7 90 unlocked) (layer "B.Fab")
+      (effects (font (size 1 1) (thickness 0.15)) (justify mirror))
+    )
+    (fp_line (start 1.8 1.4) (end 1.6 1.4) (layer "B.SilkS") (width 0.12))
+    (fp_line (start -4 0.4) (end -4 -0.4) (layer "B.SilkS") (width 0.12))
+    (fp_line (start -2.9 1.4) (end -3 1.4) (layer "B.SilkS") (width 0.12))
+    (fp_line (start 4 -0.4) (end 4 0.4) (layer "B.SilkS") (width 0.12))
+    (fp_line (start -3 -1.4) (end 2.9 -1.4) (layer "B.SilkS") (width 0.12))
+    (fp_line (start 0.4 1.4) (end -1.7 1.4) (layer "B.SilkS") (width 0.12))
+    (pad "" np_thru_hole circle (at 1.5 0 270) (size 0.85 0.85) (drill 0.85) (layers F&B.Cu *.Mask))
+    (pad "" np_thru_hole circle (at -1.5 0 270) (size 0.85 0.85) (drill 0.85) (layers F&B.Cu *.Mask))
+    (pad "1" smd roundrect (at -2.3 2.1 270) (size 1 1.5) (layers "B.Cu" "B.Paste" "B.Mask") (roundrect_rratio 0.25)
+      (net 29 "unconnected-(SW1-Pad1)") (pintype "input"))
+    (pad "2" smd roundrect (at 1 2.1 270) (size 1 1.5) (layers "B.Cu" "B.Paste" "B.Mask") (roundrect_rratio 0.25)
+      (net 9 "B+") (pintype "input"))
+    (pad "3" smd roundrect (at 2.45 2.1 270) (size 1 1.5) (layers "B.Cu" "B.Paste" "B.Mask") (roundrect_rratio 0.25)
+      (net 28 "Net-(J1-Pad2)") (pintype "input"))
+    (pad "4" smd roundrect (at 3.9 1 270) (size 1.7 1) (layers "B.Cu" "B.Paste" "B.Mask") (roundrect_rratio 0.25)
+      (net 1 "GND") (pinfunction "GND") (pintype "output"))
+    (pad "4" smd roundrect (at -4 1 270) (size 1.7 1) (layers "B.Cu" "B.Paste" "B.Mask") (roundrect_rratio 0.25)
+      (net 1 "GND") (pinfunction "GND") (pintype "output"))
+    (pad "4" smd roundrect (at 3.9 -1 270) (size 1.7 1) (layers "B.Cu" "B.Paste" "B.Mask") (roundrect_rratio 0.25)
+      (net 1 "GND") (pinfunction "GND") (pintype "output"))
+    (pad "4" smd roundrect (at -4 -1 270) (size 1.7 1) (layers "B.Cu" "B.Paste" "B.Mask") (roundrect_rratio 0.25)
+      (net 1 "GND") (pinfunction "GND") (pintype "output"))
+  )
   (gr_poly
     (pts
@@
   (via (at 192.024 63.373) (size 0.8) (drill 0.4) (layers "F.Cu" "B.Cu") (net 9))
   (segment (start 192.010331 73.66) (end 192.010331 63.386669) (width 0.508) (layer "B.Cu") (net 9))
-  (segment (start 180.32 85.350331) (end 192.010331 73.66) (width 0.508) (layer "B.Cu") (net 9))
-  (segment (start 180.32 91.0515) (end 180.32 85.350331) (width 0.508) (layer "B.Cu") (net 9))
+  (segment (start 184.43125 89.9) (end 182.5625 88.03125) (width 0.508) (layer "B.Cu") (net 9))
+  (segment (start 182.5625 88.03125) (end 182.5625 83.107831) (width 0.508) (layer "B.Cu") (net 9))
+  (segment (start 182.5625 83.107831) (end 192.010331 73.66) (width 0.508) (layer "B.Cu") (net 9))
   (segment (start 192.010331 63.386669) (end 192.024 63.373) (width 0.508) (layer "B.Cu") (net 9))
   (segment (start 133.188048 76.32796) (end 147.584592 76.32796) (width 0.381) (layer "F.Cu") (net 11))
@@
   (segment (start 173.029446 115.438651) (end 173.029446 111.846549) (width 0.254) (layer "F.Cu") (net 27))
   (segment (start 182.362002 92.765542) (end 182.362002 85.526542) (width 0.381) (layer "F.Cu") (net 27))
+  (segment (start 180.6185 91.35) (end 184.43125 91.35) (width 0.508) (layer "B.Cu") (net 28))
+  (segment (start 180.32 91.0515) (end 180.6185 91.35) (width 0.508) (layer "B.Cu") (net 28))
   (zone (net 1) (net_name "GND") (layers F&B.Cu) (hatch edge 0.508)
     (connect_pads (clearance 0.508))
