File: PCB/Diom-35SP_PCB/Diom-35SP_PCB-noSilk-black.kicad_pcb (KiCad board)
At the start: 2 copper layers, 139.9 x 113.1 mm, 38 parts, among them J1 Conn_01x02_Male, SW1 SHOU_HAN_MSK12C02-HB, U1 nice_nano

Commit message: 3d Models, New Footprints for Switches
Parts:
- MX1, MX10, MX11, MX12, MX13, MX14, MX15, MX16, MX2, MX3, MX4, MX5, MX6, MX7, MX8, MX9: footprint mx-switches-doubleSided:CherryMX-1U-doubleSided-noSilk -> hybrid-switches-DoubleSided:Kailh-V1V2-1U-doubleSided-noSilk
- MX17, MX18: footprint mx-switches-doubleSided:CherryMX-1.5U-doubleSided-Vertical-noSilk -> hybrid-switches-DoubleSided:Kailh-V1V2-1.5U-doubleSided-noSilk
- turned MX17 to 75 degrees
- turned MX18 to 65 degrees
- renumbered H18 to H17, H19 to H18
Connections:
- U1 pad 10: MX14 -> MX7
- U1 pad 12: MX7 -> MX14
Routing:
- net MX7: track 102.0 -> 77.3 mm
- net MX13: track 76.7 -> 56.7 mm
- net MX1: track 141.1 -> 148.6 mm
- net MX14: track 41.0 -> 36.0 mm
- net MX18: track 83.1 -> 78.8 mm
- net MX2: track 84.4 -> 80.3 mm
- net MX12: track 105.3 -> 109.1 mm
- net MX6: track 130.0 -> 133.5 mm
- net MX11: track 127.3 -> 130.8 mm
- net MX5: track 25.5 -> 22.1 mm
- net MX16: track 59.0 -> 56.1 mm
- net MX15: track 46.7 -> 43.8 mm
- net MX17: track 46.7 -> 44.1 mm
- net MX10: track 20.6 -> 18.4 mm
- net MX9: track 40.2 -> 38.0 mm
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- added copper zone on B.Cu, net GND
- added copper zone on F.Cu, net GND
