File: PCB/Diom-35SP_PCB/Diom-35SP_PCB.kicad_sch (KiCad schematic)
At the start: 40 parts, among them J1 Conn_01x02_Male, SW1 SHOU_HAN_MSK12C02-HB, U1 nice_nano

Commit message: Finished Renaming to 35SP
Parts:
- MX1, MX10, MX11, MX12, MX13, MX14, MX15, MX16, MX2, MX3, MX4, MX5, MX6, MX7, MX8, MX9: footprint (none) -> mx-switches-doubleSided:CherryMX-1U-doubleSided-noSilk
- MX17, MX18: footprint (none) -> mx-switches-doubleSided:CherryMX-1.5U-doubleSided-Vertical-noSilk
- gave numbers to parts that had none: 2
Changed lines of the file:
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@@
       (effects (font (size 0.508 0.508)))
     )
-    (property "Footprint" "" (id 2) (at 159.385 41.275 0)
+    (property "Footprint" "mx-switches-doubleSided:CherryMX-1U-doubleSided-noSilk" (id 2) (at 159.385 41.275 0)
       (effects (font (size 1.524 1.524)) hide)
     )
@@
       (effects (font (size 0.508 0.508)))
     )
-    (property "Footprint" "" (id 2) (at 147.955 41.275 0)
+    (property "Footprint" "mx-switches-doubleSided:CherryMX-1U-doubleSided-noSilk" (id 2) (at 147.955 41.275 0)
       (effects (font (size 1.524 1.524)) hide)
     )
@@
       (effects (font (size 0.508 0.508)))
     )
-    (property "Footprint" "" (id 2) (at 182.245 97.155 0)
+    (property "Footprint" "mx-switches-doubleSided:CherryMX-1.5U-doubleSided-Vertical-noSilk" (id 2) (at 182.245 97.155 0)
       (effects (font (size 1.524 1.524)) hide)
     )
@@
       (effects (font (size 0.508 0.508)))
     )
-    (property "Footprint" "" (id 2) (at 170.815 41.275 0)
+    (property "Footprint" "mx-switches-doubleSided:CherryMX-1U-doubleSided-noSilk" (id 2) (at 170.815 41.275 0)
       (effects (font (size 1.524 1.524)) hide)
     )
@@
       (effects (font (size 0.508 0.508)))
     )
-    (property "Footprint" "" (id 2) (at 147.955 76.835 0)
+    (property "Footprint" "mx-switches-doubleSided:CherryMX-1U-doubleSided-noSilk" (id 2) (at 147.955 76.835 0)
       (effects (font (size 1.524 1.524)) hide)
     )
@@
   (symbol (lib_id "Mechanical:MountingHole") (at 99.06 120.65 0) (unit 1)
     (in_bom yes) (on_board yes) (fields_autoplaced)
-    (property "Reference" "H?" (id 0) (at 101.6 119.3799 0)
+    (property "Reference" "H19" (id 0) (at 101.6 119.3799 0)
       (effects (font (size 1.27 1.27)) (justify left))
     )
@@
       (effects (font (size 0.508 0.508)))
     )
-    (property "Footprint" "" (id 2) (at 125.095 76.835 0)
+    (property "Footprint" "mx-switches-doubleSided:CherryMX-1U-doubleSided-noSilk" (id 2) (at 125.095 76.835 0)
       (effects (font (size 1.524 1.524)) hide)
     )
@@
       (effects (font (size 0.508 0.508)))
     )
-    (property "Footprint" "" (id 2) (at 193.675 103.505 0)
+    (property "Footprint" "mx-switches-doubleSided:CherryMX-1.5U-doubleSided-Vertical-noSilk" (id 2) (at 193.675 103.505 0)
       (effects (font (size 1.524 1.524)) hide)
     )
@@
       (effects (font (size 0.508 0.508)))
     )
-    (property "Footprint" "" (id 2) (at 170.815 97.155 0)
+    (property "Footprint" "mx-switches-doubleSided:CherryMX-1U-doubleSided-noSilk" (id 2) (at 170.815 97.155 0)
       (effects (font (size 1.524 1.524)) hide)
     )
@@
       (effects (font (size 0.508 0.508)))
     )
-    (property "Footprint" "" (id 2) (at 159.385 59.055 0)
+    (property "Footprint" "mx-switches-doubleSided:CherryMX-1U-doubleSided-noSilk" (id 2) (at 159.385 59.055 0)
       (effects (font (size 1.524 1.524)) hide)
     )
@@
   (symbol (lib_id "Mechanical:MountingHole") (at 80.01 120.65 0) (unit 1)
     (in_bom yes) (on_board yes) (fields_autoplaced)
-    (property "Reference" "H?" (id 0) (at 82.55 119.3799 0)
+    (property "Reference" "H18" (id 0) (at 82.55 119.3799 0)
       (effects (font (size 1.27 1.27)) (justify left))
     )
@@
       (effects (font (size 0.508 0.508)))
     )
-    (property "Footprint" "" (id 2) (at 147.955 59.055 0)
+    (property "Footprint" "mx-switches-doubleSided:CherryMX-1U-doubleSided-noSilk" (id 2) (at 147.955 59.055 0)
       (effects (font (size 1.524 1.524)) hide)
     )
@@
       (effects (font (size 0.508 0.508)))
     )
-    (property "Footprint" "" (id 2) (at 136.525 59.055 0)
+    (property "Footprint" "mx-switches-doubleSided:CherryMX-1U-doubleSided-noSilk" (id 2) (at 136.525 59.055 0)
       (effects (font (size 1.524 1.524)) hide)
     )
@@
       (effects (font (size 0.508 0.508)))
     )
-    (property "Footprint" "" (id 2) (at 136.525 41.275 0)
+    (property "Footprint" "mx-switches-doubleSided:CherryMX-1U-doubleSided-noSilk" (id 2) (at 136.525 41.275 0)
       (effects (font (size 1.524 1.524)) hide)
     )
@@
       (effects (font (size 0.508 0.508)))
     )
-    (property "Footprint" "" (id 2) (at 159.385 76.835 0)
+    (property "Footprint" "mx-switches-doubleSided:CherryMX-1U-doubleSided-noSilk" (id 2) (at 159.385 76.835 0)
       (effects (font (size 1.524 1.524)) hide)
     )
@@
       (effects (font (size 0.508 0.508)))
     )
-    (property "Footprint" "" (id 2) (at 170.815 59.055 0)
+    (property "Footprint" "mx-switches-doubleSided:CherryMX-1U-doubleSided-noSilk" (id 2) (at 170.815 59.055 0)
       (effects (font (size 1.524 1.524)) hide)
     )
@@
       (effects (font (size 0.508 0.508)))
     )
-    (property "Footprint" "" (id 2) (at 125.095 59.055 0)
+    (property "Footprint" "mx-switches-doubleSided:CherryMX-1U-doubleSided-noSilk" (id 2) (at 125.095 59.055 0)
       (effects (font (size 1.524 1.524)) hide)
     )
@@
       (effects (font (size 0.508 0.508)))
     )
-    (property "Footprint" "" (id 2) (at 170.815 76.835 0)
+    (property "Footprint" "mx-switches-doubleSided:CherryMX-1U-doubleSided-noSilk" (id 2) (at 170.815 76.835 0)
       (effects (font (size 1.524 1.524)) hide)
     )
@@
       (effects (font (size 0.508 0.508)))
     )
-    (property "Footprint" "" (id 2) (at 136.525 76.835 0)
+    (property "Footprint" "mx-switches-doubleSided:CherryMX-1U-doubleSided-noSilk" (id 2) (at 136.525 76.835 0)
       (effects (font (size 1.524 1.524)) hide)
     )
@@
       (effects (font (size 0.508 0.508)))
     )
-    (property "Footprint" "" (id 2) (at 125.095 41.275 0)
+    (property "Footprint" "mx-switches-doubleSided:CherryMX-1U-doubleSided-noSilk" (id 2) (at 125.095 41.275 0)
       (effects (font (size 1.524 1.524)) hide)
     )
@@
       (reference "H17") (unit 1) (value "MountingHole") (footprint "MountingHole:MountingHole_2.2mm_M2_DIN965")
     )
+    (path "/b70fb256-ccdd-4825-b06c-7fc25cd3f88f"
+      (reference "H18") (unit 1) (value "MountingHole") (footprint "MountingHole:MountingHole_2.2mm_M2_DIN965")
+    )
     (path "/4ca1e75f-3326-4617-a47f-f1d0dc149cfc"
-      (reference "H?") (unit 1) (value "MountingHole") (footprint "MountingHole:MountingHole_2.2mm_M2_DIN965")
-    )
-    (path "/b70fb256-ccdd-4825-b06c-7fc25cd3f88f"
-      (reference "H?") (unit 1) (value "MountingHole") (footprint "MountingHole:MountingHole_2.2mm_M2_DIN965")
+      (reference "H19") (unit 1) (value "MountingHole") (footprint "MountingHole:MountingHole_2.2mm_M2_DIN965")
     )
     (path "/94e4172f-7d42-4a20-80ff-c56fc225b287"

Commit message: 3d Models, New Footprints for Switches
Parts:
- removed H16, H17: MountingHole, MountingHole:MountingHole_2.2mm_M2_DIN965, symbol Mechanical:MountingHole
- MX1, MX10, MX11, MX12, MX13, MX14, MX15, MX16, MX2, MX3, MX4, MX5, MX6, MX7, MX8, MX9: footprint mx-switches-doubleSided:CherryMX-1U-doubleSided-noSilk -> (none)
- MX17, MX18: footprint mx-switches-doubleSided:CherryMX-1.5U-doubleSided-Vertical-noSilk -> (none)
- renumbered H18 to H17, H19 to H18
Connections:
- net MX14: now also U1.12 (P1.06); no longer U1.10 (P0.11)
- net MX7: now also U1.10 (P0.11); no longer U1.12 (P1.06)
Other:
- moved on the sheet: H17, H18
